File: hardware/modchip.kicad_sch (KiCad schematic)
At the start: 53 parts, among them J1 To switch T3 (I2C slave), J2 To switch T8 (GPIO46-49), J3 To switch T5 (UART0), J5 SWD, Q1 2N7002, U1 RP2350A, U2 LM66100, U5 W25Q128JVSIQ, Y1 12MHz

Commit message: hardware: title blocks name the new repository
Co-Authored-By: Claude Opus 5.5 <noreply@anthropic.com>
Claude-Session: https://claude.ai/code/session_015H5zFJRMkAr91cV6L5o8Yv
Other:
- company: github.com/wrcrooks/RTLPlayground, modchip/ -> github.com/wrcrooks/rtlplayground-modchip
Changed lines of the file:
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@@
 		(title "RTLPlayground mod chip (RP2350)")
 		(rev "A0")
-		(company "github.com/wrcrooks/RTLPlayground, modchip/")
+		(company "github.com/wrcrooks/rtlplayground-modchip")
 		(comment 1 "For SWTG024AS-V2.0 switches: management processor on headers T3, T8 and T5")
-		(comment 2 "Generated by modchip/hardware/make_sch.py; not built or tested yet")
+		(comment 2 "Generated by hardware/make_sch.py; not built or tested yet")
 	)
 	(text "POWER\nThe board runs from the switch's 3.3 V (T3/T8 pin 4) through the ideal diode U2. On the bench a debug\nprobe can supply 3.3 V on J5 pin 1 instead; U2 keeps it out of the switch. SW_SENSE tells the firmware whether\nthe switch is on: until it is, keep every switch-facing pin high-impedance with its input buffer off."
