File: hardware/modchip.kicad_pcb (KiCad board)
At the start: 4 copper layers, 106.2 x 37.2 mm, 53 parts, among them J1 To switch T3 (I2C slave), J2 To switch T8 (GPIO46-49), J3 To switch T5 (UART0), J5 SWD, Q1 2N7002, U1 RP2350A, U2 LM66100, U5 W25Q128JVSIQ, Y1 12MHz

Commit message: hardware: shorter T5 tail; production files, STL/STEP and render
The board, edited in KiCad: the tail ends about 50 mm short of T5, so the
outline is 56.95 x 37.25 mm (was 106.25 x 37.25), J3 sits at (44.5, 25.1)
mm from T3 pin 1 instead of on T5 (94.2, 24.9) and reaches T5 with a
harness, and R10/R11 moved next to it. The schematic, nets and the other
50 footprints are unchanged.

Exported from that board as saved (the scripts' placement and routing
steps not run, which would rebuild the old layout):
- production/: Gerbers and drills (zones refilled: the In1/In2 pours'
  outlines still span the old width, the fills stop 0.3 mm inside the new
  edge), BOM (unchanged), positions (R10 and R11 moved).
- mechanical/: STL and STEP without headers.
- docs/pcb-3d.png: the new board.

DRC: no errors, no unconnected items, schematic parity clean; one
warning, a dangling via on UART_RX at (136.65, 54.95) left from rerouting
J3. Checked against outline.py's obstacles: the new outline covers none
of them and keeps the U8 clip access clear.

Co-Authored-By: Claude Opus 5.5 <noreply@anthropic.com>
Claude-Session: https://claude.ai/code/session_015H5zFJRMkAr91cV6L5o8Yv
Parts:
- moved J3 49.7 mm to (136.9, 67.1)
- moved R10 48.9 mm to (133.9, 60.5), turned to -90 degrees
- moved R11 45.7 mm to (136.7, 60.5), turned to -90 degrees
Routing:
- net UART_TX: track 91.9 -> 42.8 mm
- net UART_RX: track 91.4 -> 46.5 mm, vias 0 -> 1
- net SW_U0RXD: track 4.60 -> 12.4 mm
- net SW_U0TXD: track 5.56 -> 6.22 mm
Other:
- board size 106.2 x 37.2 mm -> 56.9 x 37.2 mm
